File: pcb/pcb.kicad_pcb (KiCad board)
At the start: 2 copper layers, 50.2 x 35.6 mm, 21 parts, among them IC1 ATTINY85-P, P1 USB_OTG, P2 CONN_01X04, SW1 SW_PUSH, SW2 SW_PUSH

Commit message: Minor changes for production
Parts:
- G***: moved to B.Cu
- moved G*** 34.1 mm to (158.8, 129.3), turned to 270 degrees
Connections:
- OH1 pad 1: GND -> (no net)
- OH2 pad 1: GND -> (no net)
- OH3 pad 1: GND -> (no net)
- OH4 pad 1: GND -> (no net)
Routing:
- net GND: track 6.23 -> 12.7 mm, vias 0 -> 2
Other:
- rule trace_min: 0.2 -> 0.25
- board text added: "CYBERCOM"
- board text added: "GROUP"
- board text added: "http://www.cybercom.com"
